Commit message: Replicate kinect tf scheme.

File: softkinetic_camera/urdf/senz3d.urdf.xacro (robot description, xacro)
@@ -6,56 +6,56 @@
   <xacro:property name="M_PI" value="3.14159265359"/>
   <xacro:macro name="sensor_senz3d" params="parent name *origin">
-	<joint name="${name}_joint" type="fixed">
+    <joint name="${name}_joint" type="fixed">
       <insert_block name="origin"/>
       <parent link="${parent}"/>
-	  <child link="${name}_link"/>
-	</joint>
-	<link name="${name}_link">
-	  <visual>
-	    <origin xyz="0.0 0.0 0.0" rpy="0.0 0.0 0.0"/>
-	    <geometry>
-	      <!-- As we don't have a Senz3D mesh, use a deformed Asus Xtion Pro instead -->
-	      <mesh filename="package://softkinetic_camera/meshes/asus_xtion_pro_live.dae" scale="0.0006 0.0015 0.001"/>
-	    </geometry>
-	  </visual>
-	  <collision>
-	    <origin xyz="0.0 0.0 -0.005" rpy="0 0 0"/>
-	    <geometry>
-	    <box size="0.11 0.04 0.04"/>
-	  </geometry>
-	  </collision>
-	  <inertial>
-	    <mass value="0.271"/>
-	    <origin xyz="0 0 0"/>
-	    <inertia ixx="0.001" ixy="0.0" ixz="0.0"
-	      iyy="0.001" iyz="0.0"
-	      izz="0.001"/>
-	  </inertial>
-	</link>
-	<!-- Add frames for RGB and depth optical axes -->
-	<joint name="${name}_rgb_joint" type="fixed">
-	  <origin xyz="0.0125 0.0 0.0" rpy="0.0 0.0 0.0"/>
-	  <parent link="${name}_link"/>
-	  <child link="${name}_rgb_frame"/>
-	</joint>
-	<link name="${name}_rgb_frame"/>
-	<joint name="${name}_rgb_optical_joint" type="fixed">
-	  <origin xyz="0.0 0.0 0.0" rpy="0.0 0.0 ${M_PI}" />
-	  <parent link="${name}_rgb_frame"/>
-	  <child link="${name}_rgb_optical_frame"/>
-	</joint>
-	<link name="${name}_rgb_optical_frame"/>
-	<joint name="${name}_depth_joint" type="fixed">
-	  <origin xyz="-0.0125 0.0 0.0" rpy="0.0 0.0 0.0"/>
-	  <parent link="${name}_link"/>
-	  <child link="${name}_depth_frame"/>
-	</joint>
-	<link name="${name}_depth_frame"/>
-	<joint name="${name}_depth_optical_joint" type="fixed">
-	  <origin xyz="0.0 0.0 0.0" rpy="0.0 0.0 ${M_PI}" />
-	  <parent link="${name}_depth_frame"/>
-	  <child link="${name}_depth_optical_frame"/>
-	</joint>
-	<link name="${name}_depth_optical_frame"/>
+      <child link="${name}_link"/>
+    </joint>
+    <link name="${name}_link">
+      <visual>
+        <origin xyz="-0.01 0 0" rpy="${-M_PI/2} -${M_PI} ${-M_PI/2}"/>
+        <geometry>
+          <!-- As we don't have a Senz3D mesh, use a deformed Asus Xtion Pro instead -->
+          <mesh filename="package://softkinetic_camera/meshes/asus_xtion_pro_live.dae" scale="0.0006 0.0015 0.001"/>
+        </geometry>
+      </visual>
+      <collision>
+        <origin xyz="0.0 0.0 -0.005" rpy="0 0 0"/>
+        <geometry>
+        <box size="0.11 0.04 0.04"/>
+      </geometry>
+      </collision>
+      <inertial>
+        <mass value="0.271"/>
+        <origin xyz="0 0 0"/>
+        <inertia ixx="0.001" ixy="0.0" ixz="0.0"
+                 iyy="0.001" iyz="0.0"
+                 izz="0.001"/>
+      </inertial>
+    </link>
+    <!-- Add frames for RGB and depth optical axes -->
+    <joint name="${name}_rgb_joint" type="fixed">
+      <origin xyz="0.0 0.0125 0.0" rpy="0.0 0.0 0.0"/>
+      <parent link="${name}_link"/>
+      <child link="${name}_rgb_frame"/>
+    </joint>
+    <link name="${name}_rgb_frame"/>
+    <joint name="${name}_rgb_optical_joint" type="fixed">
+      <origin xyz="0.0 0.0 0.0" rpy="${-M_PI/2} 0.0 ${-M_PI/2}"/>
+      <parent link="${name}_rgb_frame"/>
+      <child link="${name}_rgb_optical_frame"/>
+    </joint>
+    <link name="${name}_rgb_optical_frame"/>
+    <joint name="${name}_depth_joint" type="fixed">
+      <origin xyz="0.0 -0.0125 0.0" rpy="0.0 0.0 0.0"/>
+      <parent link="${name}_link"/>
+      <child link="${name}_depth_frame"/>
+    </joint>
+    <link name="${name}_depth_frame"/>
+    <joint name="${name}_depth_optical_joint" type="fixed">
+      <origin xyz="0.0 0.0 0.0" rpy="${-M_PI/2} 0.0 ${-M_PI/2}"/>
+      <parent link="${name}_depth_frame"/>
+      <child link="${name}_depth_optical_frame"/>
+    </joint>
+    <link name="${name}_depth_optical_frame"/>
   </xacro:macro>
 </robot>

Commit message: Fix the collision box orientation. Also set realistic values for inertia , calculated with the solid cuboid formula from here: http://en.wikipedia.org/wiki/List_of_moments_of_inertia

File: softkinetic_camera/urdf/senz3d.urdf.xacro (robot description, xacro)
@@ -13,5 +13,5 @@
     <link name="${name}_link">
       <visual>
-        <origin xyz="-0.01 0 0" rpy="${-M_PI/2} -${M_PI} ${-M_PI/2}"/>
+        <origin xyz="-0.01 0.0 0.0" rpy="${-M_PI/2} -${M_PI} ${-M_PI/2}"/>
         <geometry>
           <!-- As we don't have a Senz3D mesh, use a deformed Asus Xtion Pro instead -->
@@ -20,7 +20,7 @@
       </visual>
       <collision>
-        <origin xyz="0.0 0.0 -0.005" rpy="0 0 0"/>
+        <origin xyz="-0.01 0.0 0.0" rpy="0 0 0"/>
         <geometry>
-        <box size="0.11 0.04 0.04"/>
+        <box size="0.04 0.11 0.04"/>
       </geometry>
       </collision>
@@ -28,7 +28,7 @@
         <mass value="0.271"/>
         <origin xyz="0 0 0"/>
-        <inertia ixx="0.001" ixy="0.0" ixz="0.0"
-                 iyy="0.001" iyz="0.0"
-                 izz="0.001"/>
+        <inertia ixx="0.000309392" ixy="0.0" ixz="0.0"
+                 iyy="0.000072267" iyz="0.0"
+                 izz="0.000309392"/>
       </inertial>
     </link>
